File: Hardware/Edzzanine_Console_Basic.brd (EAGLE design)
At the start: 30.5 x 44.5 mm, 25 parts, among them Q1 MOSFET-NCHANNELBSS138, Q2 MOSFET-NCHANNELBSS138, U1 MIC5219 3.3V

Commit message: finished layout, ready for review
Parts:
- removed C5, C6: 10uF, SparkFun-Capacitors:1206
- removed C7: 0.1uF, SparkFun-Capacitors:0603-CAP
- removed JP1: FTDI_DEVICE, SparkFun-Connectors:FTDI_DEVICE_SIDE
- removed Q1, Q2: MOSFET-NCHANNELBSS138, SparkFun-DiscreteSemi:SOT23
- removed R1, R2, R3, R4: 1K, SparkFun-Resistors:0603-RES
- added C1, C2: 0.1uF, SparkFun-Capacitors:0603-CAP
- added C10: 4.7uF, SparkFun-Capacitors:0603-CAP
- added C8: 10uF, SparkFun-Capacitors:1206
- added C9: 9.0pF, SparkFun-Capacitors:0603-CAP
- added FID1, FID2: FIDUCIAL1X2, SparkFun-Aesthetics:FIDUCIAL-1X2
- added JP2: (no value), SparkFun-Connectors:1X06-SMD
- added L1: (no value), SparkFun-Passives:INDUCTOR-SRP4020
- added LOGO1: SFE_LOGO_NAME_FLAME.1_INCH, SparkFun-Aesthetics:SFE_LOGO_NAME_FLAME_.1
- added LOGO4: OSHW-LOGOS, SparkFun-Aesthetics:OSHW-LOGO-S
- added R13: 680k, SparkFun-Resistors:0603-RES
- added R14: 120k, SparkFun-Resistors:0603-RES
- added U4: TPS62065, Testing:WSON-8-PAD
- U1: value MIC5219 3.3V -> (none); device SparkFun-PowerIC:SOT23-5 -> SparkFun-DigitalIC:SO14
- moved R6 11.2 mm to (19.6, 24.4)
- moved R7 6.87 mm to (19.6, 26.0), turned to 0 degrees
- moved U1 4.13 mm to (12.4, 26.4), turned to 270 degrees
- turned D3 to 0 degrees
Connections:
- removed net N$11: Q2.2, R3.1, R6.1
- removed net N$14: Q1.2, R1.1, R7.1
- new net N$18: C9.2, R13.1, R14.2, U4.4
- new net N$19: L1.P$1, U4.2
- net 1.8V: now also C2.1, U1.1; no longer Q1.1, Q2.1, R1.2, R3.2
- net GND: now also C1.2, C10.2, C2.2, C8.2, JP2.1, JP2.2, R14.1, U1.7, U1.8, U4.1, U4.3, U4.6, U4.PAD; no longer C5.2, C6.2, C7.1, JP1.P$5, JP1.P$6, U1.2
- net N$1: now also JP2.5, U1.13; no longer JP1.P$3
- net N$2: now also JP2.4, U1.12; no longer JP1.P$2
- net N$3: now also R6.1, U1.2; no longer Q1.3, R2.1
- net N$4: now also R7.1, U1.3; no longer Q2.3, R4.1
- net VCC: now also C1.1, C10.1, JP2.3, U1.14, U4.5, U4.7, U4.8; no longer C5.1, JP1.P$4, R2.2, R4.2, U1.1, U1.3
- net VSYS: now also C8.1, C9.1, L1.P$2, R13.2; no longer C6.1, C7.2, U1.5
Routing:
- net VCC: track 5.89 -> 34.3 mm, vias 0 -> 2
- net 1.8V: track 0.00 -> 23.0 mm, vias 0 -> 2
- net VSYS: track 13.1 -> 34.2 mm
- net N$3: track 0.00 -> 11.4 mm, vias 0 -> 2
- net N$4: track 0.00 -> 9.96 mm
- net N$18: track 0.00 -> 7.71 mm, vias 0 -> 2
- net N$2: track 0.00 -> 7.51 mm, vias 0 -> 2
- net N$1: track 0.00 -> 7.32 mm
- net GP135_UART_2_TX: track 14.2 -> 20.3 mm
- net N$19: track 0.00 -> 4.88 mm
- net GP134_UART_2_RX: track 8.14 -> 12.7 mm
- net PWRBTN#: track 41.2 -> 45.0 mm
- net GND: track 0.00 -> 2.25 mm, vias 2 -> 8
- net N$12: track 1.54 -> 2.36 mm
- added copper zone on layer 1, net N$18
- added copper zone on layer 1, net VCC
- added copper zone on layer 1, net VSYS
Other:
- board text added: "Console Basic Edizzanine"
- board text added: "v01"
- board text removed: "Edizzine Console"
