File: Hardware/Edzzanine_Console_Basic.sch (EAGLE design)
At the start: 25 parts, among them Q1 MOSFET-NCHANNELBSS138, Q2 MOSFET-NCHANNELBSS138, U1 MIC5219 3.3V

Commit message: finished layout, ready for review
Parts:
- removed C5, C6: 10uF, SparkFun-Capacitors:10UF-6.3V-20%(1206)
- removed C7: 0.1uF, SparkFun-Capacitors:0.1UF-25V-5%(0603)
- removed JP1: FTDI_DEVICE, SparkFun-Connectors:FTDI_DEVICE
- removed Q1, Q2: MOSFET-NCHANNELBSS138, SparkFun-DiscreteSemi:MOSFET-NCHANNELBSS138
- removed R1, R2, R3, R4: 1K, SparkFun-Resistors:1KOHM1/10W1%(0603)
- added C1, C2: 0.1uF, SparkFun-Capacitors:0.1UF-25V(+80/-20%)(0603)
- added C10: 4.7uF, SparkFun-Capacitors:4.7UF-6.3V-10%(0603)0603
- added C8: 10uF, SparkFun-Capacitors:10UF-6.3V-20%(1206)
- added C9: 9.0pF, SparkFun-Capacitors:9.0PF-50V-10%(0603)
- added FID1, FID2: FIDUCIAL1X2, SparkFun-Aesthetics:FIDUCIAL1X2
- added JP2: (no value), SparkFun-Connectors:M06SMD
- added L1: (no value), SparkFun-Passives:INDUCTOR
- added R13: 680k, SparkFun-Resistors:RESISTOR0603
- added R14: 120k, SparkFun-Resistors:RESISTOR0603
- added U4: TPS62065, Testing:TPS62065
- U1: value MIC5219 3.3V -> (none); device SparkFun-PowerIC:V_REG_MIC52193.3V -> SparkFun-DigitalIC:TXB0104PWRSOIC14
- renumbered LOGO2 to LOGO4, LOGO3 to LOGO1
Connections:
- removed net N$11: Q2.S, R3.1, R6.1
- removed net N$14: Q1.S, R1.1, R7.1
- new net N$18: C9.2, R13.1, R14.2, U4.FB
- new net N$19: L1.1, U4.SW
- net 1.8V: now also C2.1, U1.VCCA; no longer Q1.G, Q2.G, R1.2, R3.2
- net GND: now also C1.2, C10.2, C2.2, C8.2, JP2.1, JP2.2, R14.1, U1.OE, U4.AGND, U4.PAD, U4.PG, U4.PGND; no longer C5.2, C6.2, C7.1, JP1.CTS, JP1.GND
- net N$1: now also JP2.5, U1.B1; no longer JP1.RXI
- net N$2: now also JP2.4, U1.B2; no longer JP1.TXO
- net N$3: now also R6.1, U1.A1; no longer Q1.D, R2.1
- net N$4: now also R7.1, U1.A2; no longer Q2.D, R4.1
- net VCC: now also C1.1, C10.1, JP2.3, U1.VCCB, U4.AVIN, U4.EN, U4.PVIN; no longer C5.1, JP1.VCC, R2.2, R4.2, U1.EN, U1.IN
- net VSYS: now also C8.1, C9.1, L1.2, R13.2; no longer C6.1, C7.2, U1.OUT
