File: Hardware/Edzzanine_Console_Basic.sch (EAGLE design)
At the start: 27 parts, among them U4 TPS62065

Commit message: fixed rx tx
Connections:
- net N$1 renamed RXD
- net N$2 renamed TXD
- net N$3: now also R7.1; no longer R6.1
- net N$4: now also R6.1; no longer R7.1
Other:
- note added: "Black"
- note added: "Green"
- moved on the sheet: R6, R7
Changed lines of the file:
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@@
 <sheet>
 <plain>
+<text x="30.48" y="114.3" size="1.778" layer="94">Black</text>
+<text x="30.48" y="132.08" size="1.778" layer="94">Green</text>
 </plain>
 <instances>
@@
 <attribute name="NAME" x="223.52" y="104.14" size="1.778" layer="95" rot="R90"/>
 </instance>
-<instance part="R6" gate="G$1" x="93.98" y="127" smashed="yes">
-<attribute name="NAME" x="90.17" y="128.4986" size="1.778" layer="95"/>
-<attribute name="VALUE" x="95.25" y="128.778" size="1.778" layer="96"/>
+<instance part="R6" gate="G$1" x="91.44" y="124.46" smashed="yes" rot="MR180">
+<attribute name="NAME" x="87.63" y="122.9614" size="1.778" layer="95" rot="MR180"/>
+<attribute name="VALUE" x="92.71" y="122.682" size="1.778" layer="96" rot="MR180"/>
 </instance>
-<instance part="R7" gate="G$1" x="93.98" y="124.46" smashed="yes">
-<attribute name="NAME" x="90.17" y="120.8786" size="1.778" layer="95"/>
-<attribute name="VALUE" x="95.25" y="121.158" size="1.778" layer="96"/>
+<instance part="R7" gate="G$1" x="91.44" y="127" smashed="yes" rot="MR180">
+<attribute name="NAME" x="87.63" y="130.5814" size="1.778" layer="95" rot="MR180"/>
+<attribute name="VALUE" x="92.71" y="130.302" size="1.778" layer="96" rot="MR180"/>
 </instance>
 <instance part="S1" gate="G$1" x="78.74" y="53.34"/>
@@
 <segment>
 <pinref part="R7" gate="G$1" pin="2"/>
-<wire x1="99.06" y1="124.46" x2="104.14" y2="124.46" width="0.1524" layer="91"/>
+<wire x1="96.52" y1="127" x2="104.14" y2="127" width="0.1524" layer="91"/>
+<label x="104.14" y="127" size="1.27" layer="95" xref="yes"/>
+</segment>
+</net>
+<net name="GP134_UART_2_RX" class="0">
+<segment>
+<pinref part="R6" gate="G$1" pin="2"/>
+<wire x1="96.52" y1="124.46" x2="104.14" y2="124.46" width="0.1524" layer="91"/>
 <label x="104.14" y="124.46" size="1.27" layer="95" xref="yes"/>
-</segment>
-</net>
-<net name="GP134_UART_2_RX" class="0">
-<segment>
-<pinref part="R6" gate="G$1" pin="2"/>
-<wire x1="99.06" y1="127" x2="104.14" y2="127" width="0.1524" layer="91"/>
-<label x="104.14" y="127" size="1.27" layer="95" xref="yes"/>
 </segment>
 </net>
@@
 </segment>
 </net>
-<net name="N$1" class="0">
+<net name="RXD" class="0">
 <segment>
 <pinref part="U1" gate="G$1" pin="B1"/>
 <wire x1="33.02" y1="127" x2="50.8" y2="127" width="0.1524" layer="91"/>
 <pinref part="JP2" gate="G$1" pin="5"/>
-</segment>
-</net>
-<net name="N$2" class="0">
+<label x="40.64" y="127" size="1.778" layer="95"/>
+</segment>
+</net>
+<net name="TXD" class="0">
 <segment>
 <pinref part="U1" gate="G$1" pin="B2"/>
 <wire x1="50.8" y1="124.46" x2="33.02" y2="124.46" width="0.1524" layer="91"/>
 <pinref part="JP2" gate="G$1" pin="4"/>
+<label x="40.64" y="124.46" size="1.778" layer="95"/>
 </segment>
 </net>
@@
 <segment>
 <pinref part="U1" gate="G$1" pin="A1"/>
+<wire x1="86.36" y1="127" x2="81.28" y2="127" width="0.1524" layer="91"/>
+<pinref part="R7" gate="G$1" pin="1"/>
+</segment>
+</net>
+<net name="N$4" class="0">
+<segment>
+<pinref part="U1" gate="G$1" pin="A2"/>
+<wire x1="86.36" y1="124.46" x2="81.28" y2="124.46" width="0.1524" layer="91"/>
 <pinref part="R6" gate="G$1" pin="1"/>
-<wire x1="88.9" y1="127" x2="81.28" y2="127" width="0.1524" layer="91"/>
-</segment>
-</net>
-<net name="N$4" class="0">
-<segment>
-<pinref part="U1" gate="G$1" pin="A2"/>
-<pinref part="R7" gate="G$1" pin="1"/>
-<wire x1="88.9" y1="124.46" x2="81.28" y2="124.46" width="0.1524" layer="91"/>
-</segment>
-</net>
+</segment>
+</net>

Commit message: fixed OE to high
Connections:
- net 1.8V: now also U1.OE
- net GND: no longer U1.OE
Changed lines of the file:
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@@
 <part name="SUPPLY2" library="SparkFun-Aesthetics" deviceset="VCC" device=""/>
 <part name="GND2" library="SparkFun-Aesthetics" deviceset="GND" device=""/>
-<part name="GND5" library="SparkFun-Aesthetics" deviceset="GND" device=""/>
 <part name="SUPPLY3" library="SparkFun-Aesthetics" deviceset="VCC" device=""/>
 <part name="SUPPLY4" library="SparkFun-Aesthetics" deviceset="VCC" device=""/>
@@
 <part name="SUPPLY6" library="SparkFun-Aesthetics" deviceset="VCC" device=""/>
 <part name="SUPPLY7" library="SparkFun-Aesthetics" deviceset="1.8V" device=""/>
+<part name="SUPPLY8" library="SparkFun-Aesthetics" deviceset="1.8V" device=""/>
 </parts>
 <sheets>
@@
 <instance part="SUPPLY2" gate="G$1" x="63.5" y="144.78"/>
 <instance part="GND2" gate="1" x="66.04" y="106.68"/>
-<instance part="GND5" gate="1" x="83.82" y="106.68"/>
 <instance part="SUPPLY3" gate="G$1" x="139.7" y="139.7"/>
 <instance part="SUPPLY4" gate="G$1" x="147.32" y="139.7"/>
@@
 <instance part="SUPPLY6" gate="G$1" x="15.24" y="129.54"/>
 <instance part="SUPPLY7" gate="G$1" x="129.54" y="129.54"/>
+<instance part="SUPPLY8" gate="G$1" x="83.82" y="132.08"/>
 </instances>
 <busses>
@@
 <pinref part="U1" gate="G$1" pin="GND"/>
 <pinref part="GND2" gate="1" pin="GND"/>
-</segment>
-<segment>
-<pinref part="U1" gate="G$1" pin="OE"/>
-<wire x1="81.28" y1="132.08" x2="83.82" y2="132.08" width="0.1524" layer="91"/>
-<wire x1="83.82" y1="132.08" x2="83.82" y2="109.22" width="0.1524" layer="91"/>
-<pinref part="GND5" gate="1" pin="GND"/>
 </segment>
 <segment>
@@
 <pinref part="SUPPLY7" gate="G$1" pin="1.8V"/>
 </segment>
-</net>
+<segment>
+<pinref part="U1" gate="G$1" pin="OE"/>
+<wire x1="81.28" y1="132.08" x2="83.82" y2="132.08" width="0.1524" layer="91"/>
+<pinref part="SUPPLY8" gate="G$1" pin="1.8V"/>
+</segment>
+</net>
